File: Hardware/Estação/Placa Mãe/Dev_1.2/RiMon.kicad_sch (KiCad schematic)
At the start: 55 parts, among them J1 5vEx, J2 IO, J3 PGM2, J4 USS, J5 LCD, J6 SNS_PWR, J7 USB_B_Micro, J8 Pluv, J9 Lidar, Q1 SS8050-G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

Commit message: Progresso alterações
Parts:
- removed D1: BAT760-7, Diode_SMD:D_SOD-323_HandSoldering, symbol Device:D_Schottky
- removed J7: USB_B_Micro, Connector_USB:USB_Micro-B_GCT_USB3076-30-A, symbol Connector:USB_B_Micro
- removed Q1, Q2: SS8050-G, Package_TO_SOT_SMD:SOT-23, symbol Device:Q_NPN_BEC
- removed U4: CP2102N, Package_DFN_QFN:QFN-24-1EP_4x4mm_P0.5mm_EP2.6x2.6mm, symbol Interface_USB:CP2102N-Axx-xQFN24
- added C17: 22nF, Capacitor_SMD:C_0805_2012Metric_Pad1.18x1.45mm_HandSolder, symbol Device:C
- added C18, C21: 100nF, Capacitor_SMD:C_0805_2012Metric_Pad1.18x1.45mm_HandSolder, symbol Device:C
- added C22, C23: 22uF, Capacitor_SMD:C_1206_3216Metric_Pad1.33x1.80mm_HandSolder, symbol Device:C
- added C24: 300pF, Capacitor_SMD:C_0805_2012Metric_Pad1.18x1.45mm_HandSolder, symbol Device:C
- added L1: 6.8uH, Inductor_SMD:L_Wuerth_HCI-1040, symbol Device:L
- added U4: MP2338GTL, Package_TO_SOT_SMD:SOT-583-8, symbol Regulator_Switching:MP2338GTL
- C11: value 4.7uF -> 22uF
- C12: value 100nF -> 22uF; footprint Capacitor_SMD:C_0805_2012Metric_Pad1.18x1.45mm_HandSolder -> Capacitor_SMD:C_1206_3216Metric_Pad1.33x1.80mm_HandSolder
- J1: value 5vEx -> PWR; footprint TerminalBlock_Phoenix:TerminalBlock_Phoenix_MKDS-1,5-2-5.08_1x02_P5.08mm_Horizontal -> TerminalBlock_Phoenix:TerminalBlock_Phoenix_MKDS-1,5-3-5.08_1x03_P5.08mm_Horizontal; symbol Connector:Conn_01x02_Socket -> Connector:Conn_01x03_Socket
- R4: value 2k -> 191k
- R5: value 10k -> 50k
- R7: value 22k1 -> 10k
- R8: value 10k -> 91k
- R9: value 47k5 -> 10k
- SW1, SW2: footprint Button_Switch_SMD:SW_Push_1P1T_NO_CK_KMR2 -> Button_Switch_SMD:SW_Push_1P1T_NO_6x6mm_H9.5mm
- U5: footprint Package_SO:SOP-4_3.8x4.1mm_P2.54mm -> Package_SO:SSO-4_6.7x5.1mm_P2.54mm_Clearance8mm
Connections:
- net UART_SUSPEND is gone; now on an unnamed net: R8.1
- net USB_VBUS is gone; now on an unnamed net: R7.1
- net +3.3V: now also J4.1 (Pin_1); no longer C12.1, R4.2
- net +5V: now also J1.2 (Pin_2), R8.2, R9.2, C22.1, C23.1, C24.2, L1.2; no longer J1.1 (Pin_1), J4.1 (Pin_1)
- net GND: now also J1.3 (Pin_3), R5.2, R7.2, C17.2, C18.2, C22.2, C23.2, U4.4 (GND); no longer J1.2 (Pin_2), R8.2, R9.2
- net at R6.2: now also C24.1
- net +12V: now reaches R4.1
- net +12V: now also C12.1, J1.1 (Pin_1), C18.1, U4.2 (IN)
- net DTR: no longer names the net of R5.1
- net DTR: now also R4.2, U4.6 (EN)
- net RTS: no longer names the net of R6.1
- net RTS: now also U4.8 (FB)
- net VBUS_DIV: no longer names the net of R9.1
- net VBUS_DIV: now also U4.1 (PG); no longer R7.2
- new net: C21.2, L1.1, U4.3 (SW)
- new net: C21.1, U4.5 (BST)
- new net: C17.1, U4.7 (SS)
- no-connect marks 19 -> 9
Other:
- note added: "BUCK Converter"
- note removed: "USB/UART"
