File: Hardware/Estação/Placa Mãe/Dev_1.2/RiMon.kicad_pcb (KiCad board)
At the start: 4 copper layers, 63.2 x 42.9 mm, 55 parts, among them J1 5vEx, J2 IO, J3 PGM2, J4 USS, J5 LCD, J6 SNS_PWR, J7 USB_B_Micro, J8 Pluv, J9 Lidar, Q1 SS8050-G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

Commit message: Progresso alterações
Parts:
- removed D1: BAT760-7, Diode_SMD:D_SOD-323_HandSoldering
- removed J7: USB_B_Micro, Connector_USB:USB_Micro-B_GCT_USB3076-30-A
- removed Q1, Q2: SS8050-G, Package_TO_SOT_SMD:SOT-23
- added C17: 22nF, Capacitor_SMD:C_0805_2012Metric_Pad1.18x1.45mm_HandSolder, F.Cu at (100.2, 119.9)
- added C18: 100nF, Capacitor_SMD:C_0805_2012Metric_Pad1.18x1.45mm_HandSolder, B.Cu at (105.4, 111.3)
- added C21: 100nF, Capacitor_SMD:C_0805_2012Metric_Pad1.18x1.45mm_HandSolder, F.Cu at (110.0, 118.5)
- added C22: 22uF, Capacitor_SMD:C_1206_3216Metric_Pad1.33x1.80mm_HandSolder, B.Cu at (110.2, 111.3)
- added C23: 22uF, Capacitor_SMD:C_1206_3216Metric_Pad1.33x1.80mm_HandSolder, B.Cu at (107.8, 111.3)
- added C24: 300pF, Capacitor_SMD:C_0805_2012Metric_Pad1.18x1.45mm_HandSolder, F.Cu at (100.2, 124.1)
- added L1: 6.8uH, Inductor_SMD:L_Wuerth_HCI-1040, F.Cu at (106.5, 111.3)
- C10, C9, U2: moved to B.Cu
- C11: value 4.7uF -> 22uF; moved to B.Cu
- C12: value 100nF -> 22uF; footprint Capacitor_SMD:C_0805_2012Metric_Pad1.18x1.45mm_HandSolder -> Capacitor_SMD:C_1206_3216Metric_Pad1.33x1.80mm_HandSolder; moved to B.Cu
- J1: value 5vEx -> PWR; footprint TerminalBlock_Phoenix:TerminalBlock_Phoenix_MKDS-1,5-2-5.08_1x02_P5.08mm_Horizontal -> TerminalBlock_Phoenix:TerminalBlock_Phoenix_MKDS-1,5-3-5.08_1x03_P5.08mm_Horizontal
- J4: moved to F.Cu
- R4: value 2k -> 191k
- R5: value 10k -> 50k
- R7: value 22k1 -> 10k
- R8: value 10k -> 91k
- R9: value 47k5 -> 10k
- SW1, SW2: footprint Button_Switch_SMD:SW_Push_1P1T_NO_CK_KMR2 -> Button_Switch_SMD:SW_Push_1P1T_NO_6x6mm_H9.5mm
- U4: value CP2102N -> MP2338GTL; footprint Package_DFN_QFN:QFN-24-1EP_4x4mm_P0.5mm_EP2.6x2.6mm -> Package_TO_SOT_SMD:SOT-583-8; moved to F.Cu
- U5: footprint Package_SO:SOP-4_3.8x4.1mm_P2.54mm -> Package_SO:SSO-4_6.7x5.1mm_P2.54mm_Clearance8mm
- moved SW1 43.2 mm to (131.6, 124.0)
- moved J4 19.2 mm to (116.0, 123.9)
- moved C11 18.5 mm to (115.0, 126.2)
- moved R8 18.0 mm to (100.2, 126.2), turned to 180 degrees
- moved R7 15.1 mm to (100.2, 121.9)
- moved R4 15.1 mm to (111.8, 124.8)
- moved R5 13.4 mm to (109.9, 124.8)
- moved R9 9.82 mm to (99.9, 114.6), turned to 90 degrees
- moved U4 9.21 mm to (110.4, 121.1), turned to 180 degrees
- moved SW2 9.16 mm to (142.6, 124.0), turned to 0 degrees
- moved C2 8.63 mm to (107.4, 103.0), turned to 90 degrees
- moved C12 7.23 mm to (103.3, 111.3), turned to 90 degrees
- moved R6 5.39 mm to (107.1, 120.8)
- moved U2 4.19 mm to (108.7, 102.8), turned to 90 degrees
- moved C3 4.19 mm to (110.0, 103.0), turned to -90 degrees
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Connections:
- C12 pad 1: +3.3V -> +12V
- J1 pad 1: +5V -> +12V
- J1 pad 2: GND -> +5V
- J4 pad 1: +5V -> +3.3V
- R4 pad 1: Net-(U4-~{RST}) -> +12V
- R4 pad 2: +3.3V -> Net-(U4-EN)
- R5 pad 1: /DTR -> Net-(U4-EN)
- R5 pad 2: Net-(Q1-B) -> GND
- R6 pad 1: /RTS -> Net-(U4-FB)
- R6 pad 2: Net-(Q2-B) -> Net-(C24-Pad1)
- R7 pad 1: /USB_VBUS -> Net-(C24-Pad1)
- R7 pad 2: /VBUS_DIV -> GND
- R8 pad 1: /UART_SUSPEND -> Net-(C24-Pad1)
- R8 pad 2: GND -> +5V
- R9 pad 1: /VBUS_DIV -> Net-(U4-PG)
- R9 pad 2: GND -> +5V
- U4 pad 1: unconnected-(U4-~{RI}/CLK-Pad1) -> Net-(U4-PG)
- U4 pad 2: GND -> +12V
- U4 pad 3: /USB_DP -> Net-(U4-SW)
- U4 pad 4: /USB_DN -> GND
- U4 pad 5: +3.3V -> Net-(U4-BST)
- U4 pad 6: +3.3V -> Net-(U4-EN)
- U4 pad 7: +3.3V -> Net-(U4-SS)
- U4 pad 8: /VBUS_DIV -> Net-(U4-FB)
Routing:
- net +3.3V: track 192.5 -> 22.1 mm, vias 18 -> 1
- net /EN: track 91.7 -> 0.00 mm, vias 2 -> 0
- net /IO0: track 54.9 -> 0.00 mm, vias 2 -> 0
- net /IO04: track 51.0 -> 0.00 mm, vias 2 -> 0
- net +12V: track 0.00 -> 49.2 mm, vias 0 -> 1
- net /TXD0: track 46.4 -> 0.00 mm
- net /RXD0: track 45.9 -> 0.00 mm
- net /L_TXD: track 38.7 -> 0.00 mm, vias 2 -> 0
- net /L_RXD: track 38.4 -> 0.00 mm, vias 2 -> 0
- net /SX_RST: track 38.2 -> 0.00 mm, vias 2 -> 0
- net /LCD_SCK: track 35.6 -> 0.00 mm
- net /LCD_SDA: track 32.6 -> 0.00 mm
- net /SX_DIO2: track 29.0 -> 0.00 mm, vias 2 -> 0
- net /SX_SCK: track 27.4 -> 0.00 mm, vias 2 -> 0
- net /SX_MOSI: track 27.3 -> 0.00 mm
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- removed copper zone on In2.Cu, net +3.3V
Other:
- board size 63.2 x 42.9 mm -> 63.2 x 49.3 mm
- board text added: "3v3 RX TX GND"
- board text added: "GND +5v +12v"
- board text removed: "GND +5v"

Commit message: Finaliza traces v1.2
Parts:
- moved R2 14.5 mm to (145.4, 97.3), turned to 90 degrees
- moved R3 12.1 mm to (143.4, 97.3), turned to -90 degrees
- moved SW1 11.0 mm to (142.6, 123.7)
- moved SW2 10.9 mm to (131.7, 123.7)
- moved C13 10.7 mm to (141.4, 97.3), turned to 90 degrees
- moved J6 0.25 mm to (110.7, 91.2)
- moved J8 0.25 mm to (127.8, 83.6)
- moved R12 0.11 mm to (117.7, 86.9), turned to 0 degrees
Routing:
- net +3.3V: track 22.1 -> 192.9 mm, vias 1 -> 3
- net /IO04: track 0.00 -> 64.2 mm, vias 0 -> 1
- net /L_RXD: track 0.00 -> 58.1 mm, vias 0 -> 1
- net /L_TXD: track 0.00 -> 54.7 mm, vias 0 -> 1
- net /IO0: track 0.00 -> 52.5 mm, vias 0 -> 2
- net /EN: track 0.00 -> 47.3 mm, vias 0 -> 2
- net /SX_RST: track 0.00 -> 44.8 mm, vias 0 -> 2
- net /LCD_SCK: track 0.00 -> 34.6 mm, vias 0 -> 1
- net +5V: track 79.2 -> 110.6 mm
- net /LCD_SDA: track 0.00 -> 28.0 mm, vias 0 -> 1
- net /SX_DIO2: track 0.00 -> 27.7 mm, vias 0 -> 2
- net /SX_MOSI: track 0.00 -> 27.0 mm, vias 0 -> 2
- net Net-(R10-Pad1): track 0.00 -> 25.3 mm, vias 0 -> 1
- net /DX_DIO1: track 0.00 -> 24.0 mm, vias 0 -> 2
- net /VBAT: track 0.00 -> 21.7 mm
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