File: Hardware/Estação/Placa Mãe/Dev_1.3/RiMon.kicad_sch (KiCad schematic)
At the start: 56 parts, among them J1 PWR, J2 IO, J3 PGM2, J4 USS, J5 LCD, J6 SNS_PWR, J7 Radio, J8 Pluv, J9 Lidar, SW1 EN, SW2 IO0, U1 ESP32-WROOM-32, U2 AMS1117, U4 MP2338GTL, U5 PC817

Commit message: v1.3 conectado e organizado
Parts:
- added J4: JBAT, Connector_PinSocket_2.54mm:PinSocket_1x02_P2.54mm_Vertical, symbol Connector:Conn_01x02_Socket
- added J6: I2C, Connector_PinSocket_2.54mm:PinSocket_1x04_P2.54mm_Vertical, symbol Connector:Conn_01x04_Socket
- D1: renamed from D3; footprint LED_SMD:LED_0805_2012Metric_Pad1.15x1.40mm_HandSolder -> LED_THT:LED_D3.0mm
- D2: footprint LED_SMD:LED_0805_2012Metric_Pad1.15x1.40mm_HandSolder -> LED_THT:LED_D3.0mm
- D3: renamed from D4; footprint LED_SMD:LED_0805_2012Metric_Pad1.15x1.40mm_HandSolder -> LED_THT:LED_D3.0mm
- renumbered C6 to C10, C4 to C11, C13 to C12, C5 to C13, C19 to C14, C10 to C15, C20 to C16, C11 to C17, C9 to C18, C22 to C19, C3 to C2, C18 to C20, C23 to C21, C12 to C22, C2 to C3, C17 to C4, C21 to C5, C24 to C6, C16 to C7, C14 to C8, C15 to C9, J2 to J10, J3 to J11, J6 to J2, J8 to J3, J7 to J5, J5 to J7, J4 to J8, R8 to R1, R12 to R10, R10 to R11, R11 to R12, R9 to R2, R6 to R3, R5 to R4, R4 to R5, R7 to R6, R1 to R7, R3 to R8, R2 to R9, SW2 to SW1, SW1 to SW2, U5 to U2, U4 to U3, U2 to U4
Connections:
- net +12V: now also J4.1 (Pin_1); no longer J10.6 (Pin_6), R9.1
- net +3.3V: now also J6.1 (Pin_1)
- net GND: now also J6.3 (Pin_3)
- net LCD_SCK: now also J6.4 (Pin_4)
- net LCD_SDA: now also J6.2 (Pin_2)
- new net VBAT: J4.2 (Pin_2), R9.1
Other:
- note added: "LCD/I2C"
- note removed: "LCD"
- moved on the sheet: C15, C18, J10, J11, J2, J5, J7
