File: Hardware/Estação/Placa Mãe/Dev_1.3/RiMon.kicad_sch (KiCad schematic)
At the start: 58 parts, among them J1 PWR, J10 IO, J11 PGM2, J2 SNS_PWR, J3 Pluv, J4 JBAT, J5 Radio, J6 I2C, J7 LCD, J8 USS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

Commit message: Limpeza geral
Parts:
- renumbered D3 to D1, D1 to D3
Connections:
- net L_RXD renamed U2_TX
- net L_TXD renamed U2_RX
Changed lines of the file:
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@@
 	(wire
 		(pts
-			(xy 163.83 184.15) (xy 166.37 184.15)
-		)
-		(stroke
-			(width 0)
-			(type default)
-		)
-	)
-	(wire
-		(pts
 			(xy 58.42 38.1) (xy 58.42 43.18)
 		)
@@
 	(wire
 		(pts
-			(xy 163.83 186.69) (xy 166.37 186.69)
-		)
-		(stroke
-			(width 0)
-			(type default)
-		)
-	)
-	(wire
-		(pts
 			(xy 184.15 109.22) (xy 182.88 109.22)
 		)
@@
 	)
 	(label "U2_TX"
-		(at 166.37 184.15 0)
+		(at 146.05 158.75 0)
 		(fields_autoplaced yes)
 		(effects
@@
 		)
 	)
+	(label "U2_RX"
+		(at 146.05 161.29 0)
+		(fields_autoplaced yes)
+		(effects
+			(font
+				(size 1.27 1.27)
+			)
+			(justify left bottom)
+		)
+	)
 	(label "HSPI_CLK"
 		(at 162.56 140.97 0)
@@
 		)
 	)
-	(label "L_RXD"
-		(at 163.83 184.15 180)
+	(label "U2_TX"
+		(at 146.05 180.34 0)
 		(fields_autoplaced yes)
 		(effects
@@
 				(size 1.27 1.27)
 			)
-			(justify right bottom)
+			(justify left bottom)
 		)
 	)
@@
 		)
 	)
-	(label "L_RXD"
-		(at 146.05 180.34 0)
-		(fields_autoplaced yes)
-		(effects
-			(font
-				(size 1.27 1.27)
-			)
-			(justify left bottom)
-		)
-	)
 	(label "tmpGND"
 		(at 146.05 107.95 180)
@@
 	)
 	(label "U2_RX"
-		(at 166.37 186.69 0)
+		(at 146.05 182.88 0)
 		(fields_autoplaced yes)
 		(effects
@@
 		)
 	)
-	(label "L_TXD"
-		(at 146.05 182.88 0)
-		(fields_autoplaced yes)
-		(effects
-			(font
-				(size 1.27 1.27)
-			)
-			(justify left bottom)
-		)
-	)
 	(label "RXD0"
 		(at 161.29 113.03 0)
@@
 		)
 	)
-	(label "L_TXD"
-		(at 163.83 186.69 180)
-		(fields_autoplaced yes)
-		(effects
-			(font
-				(size 1.27 1.27)
-			)
-			(justify right bottom)
-		)
-	)
 	(label "SX_DIO2"
 		(at 60.96 170.18 0)
@@
 		)
 	)
-	(label "L_TXD"
-		(at 146.05 161.29 0)
-		(fields_autoplaced yes)
-		(effects
-			(font
-				(size 1.27 1.27)
-			)
-			(justify left bottom)
-		)
-	)
 	(label "IO34"
 		(at 162.56 135.89 0)
@@
 		)
 	)
-	(label "L_RXD"
-		(at 146.05 158.75 0)
-		(fields_autoplaced yes)
-		(effects
-			(font
-				(size 1.27 1.27)
-			)
-			(justify left bottom)
-		)
-	)
 	(label "HSPI_MISO"
 		(at 60.96 134.62 0)
@@
 		(on_board yes)
 		(dnp no)
-		(property "Reference" "D1"
+		(property "Reference" "D3"
 			(at 233.426 136.144 0)
 			(effects
@@
 			(project "RiMon"
 				(path "/6cdf9bd6-c189-4ca4-a68f-3d1947227cf7"
-					(reference "D1")
+					(reference "D3")
 					(unit 1)
 				)
@@
 		(on_board yes)
 		(dnp no)
-		(property "Reference" "D3"
+		(property "Reference" "D1"
 			(at 233.426 141.224 0)
 			(effects
@@
 			(project "RiMon"
 				(path "/6cdf9bd6-c189-4ca4-a68f-3d1947227cf7"
-					(reference "D3")
+					(reference "D1")
 					(unit 1)
 				)
@@
 		(dnp no)
 		(property "Reference" "R3"
-			(at 194.31 64.77 0)
+			(at 195.326 64.008 90)
 			(effects
 				(font
@@
 		)
 		(property "Value" "10k"
-			(at 196.596 65.024 0)
+			(at 197.358 66.04 90)
 			(effects
 				(font
@@
 		(dnp no)
 		(property "Reference" "R2"
-			(at 194.31 59.69 0)
+			(at 195.326 58.928 90)
 			(effects
 				(font
@@
 		)
 		(property "Value" "10k"
-			(at 196.596 59.69 0)
+			(at 197.358 60.96 90)
 			(effects
 				(font

Commit message: Ajustes fabricação
Connections:
- net GND: now also J10.6 (Pin_6)
Changed lines of the file:
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@@
+		)
+	)
+	(label "tmpGND"
+		(at 147.32 138.43 180)
+		(fields_autoplaced yes)
+		(effects
+			(font
+				(size 1.27 1.27)
+			)
+			(justify right bottom)
 		)
 	)
