File: Hardware/Estação/Placa Mãe/Dev_1.3/RiMon.kicad_pcb (KiCad board)
At the start: 4 copper layers, 63.2 x 49.3 mm, 56 parts, among them J1 PWR, J2 IO, J3 PGM2, J4 USS, J5 LCD, J6 SNS_PWR, J7 Radio, J8 Pluv, J9 Lidar, SW1 EN, SW2 IO0, U1 ESP32-WROOM-32, U2 AMS1117, U4 MP2338GTL, U5 PC817

Commit message: v1.3 conectado e organizado
Parts:
- added J4: JBAT, Connector_PinSocket_2.54mm:PinSocket_1x02_P2.54mm_Vertical, F.Cu at (114.4, 91.2)
- added J6: I2C, Connector_PinSocket_2.54mm:PinSocket_1x04_P2.54mm_Vertical, F.Cu at (115.6, 113.0)
- D1: renamed from D3; footprint LED_SMD:LED_0805_2012Metric_Pad1.15x1.40mm_HandSolder -> LED_THT:LED_D3.0mm
- D2: footprint LED_SMD:LED_0805_2012Metric_Pad1.15x1.40mm_HandSolder -> LED_THT:LED_D3.0mm
- D3: renamed from D4; footprint LED_SMD:LED_0805_2012Metric_Pad1.15x1.40mm_HandSolder -> LED_THT:LED_D3.0mm
- moved D3 17.6 mm to (121.8, 96.6), turned to 180 degrees
- moved R14 15.2 mm to (116.2, 101.2), turned to 180 degrees
- moved R15 13.8 mm to (116.3, 96.6), turned to 180 degrees
- moved D1 13.7 mm to (121.8, 101.2), turned to 180 degrees
- moved R13 12.3 mm to (116.3, 105.8), turned to 180 degrees
- moved D2 9.37 mm to (121.8, 105.8), turned to 180 degrees
- moved C17 5.53 mm to (116.6, 120.9), turned to 0 degrees
- moved C15 5.17 mm to (116.6, 110.7), turned to 180 degrees
- moved C18 2.84 mm to (119.1, 115.8), turned to 0 degrees
- moved J8 0.85 mm to (115.6, 123.2)
- moved J7 0.63 mm to (115.6, 118.1)
- renumbered C6 to C10, C4 to C11, C13 to C12, C5 to C13, C19 to C14, C10 to C15, C20 to C16, C11 to C17, C9 to C18, C22 to C19, C3 to C2, C18 to C20, C23 to C21, C12 to C22, C2 to C3, C17 to C4, C21 to C5, C24 to C6, C16 to C7, C14 to C8, C15 to C9, J2 to J10, J3 to J11, J6 to J2, J8 to J3, J7 to J5, J5 to J7, J4 to J8, R8 to R1, R12 to R10, R10 to R11, R11 to R12, R9 to R2, R6 to R3, R5 to R4, R4 to R5, R7 to R6, R1 to R7, R3 to R8, R2 to R9, SW2 to SW1, SW1 to SW2, U5 to U2, U4 to U3, U2 to U4
Connections:
- J10 pad 6: +12V -> unconnected-(J10-Pin_6-Pad6)
- R9 pad 1: +12V -> /VBAT
Routing:
- net +3.3V: track 46.2 -> 155.0 mm, vias 2 -> 3
- net +5V: track 80.1 -> 127.9 mm
- net /VBAT: track 0.00 -> 29.1 mm, vias 0 -> 1
- net /IO0: track 49.9 -> 62.2 mm
- net /LCD_SDA: track 25.9 -> 37.8 mm
- net /LED_Status: track 17.0 -> 22.9 mm
- net +12V: track 60.8 -> 63.8 mm
- net /IO04: track 65.3 -> 62.4 mm
- net /EN: track 46.9 -> 49.2 mm, vias 1 -> 2
- net Net-(D1-A): track 0.00 -> 2.03 mm
- net Net-(D2-A): track 0.00 -> 1.91 mm
- net /LCD_SCK: track 31.5 -> 33.1 mm
- net Net-(D3-A): track 2.67 -> 1.91 mm, vias 1 -> 0
- net /L_RXD: track 27.1 -> 27.9 mm
- net /L_TXD: track 23.5 -> 24.2 mm
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- added copper zone on In2.Cu, net GND
Other:
- board text added: "3v3 SDA GND SCK"
- board text added: "GND DHT Pluv 3.3v"
- board text added: "I2C"
- board text added: "Rádio"

Commit message: Limpeza geral
Parts:
- moved C9 0.51 mm to (146.8, 83.8)
- renumbered D3 to D1, D1 to D3
Connections:
- net /L_RXD renamed /U2_TX
- net /L_TXD renamed /U2_RX
Other:
- board text added: "5v XMI XMO XIO1 XIO0"
- board text added: "XNS XSC XRS XIO2 GND"
Changed lines of the file:
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@@
 	(net 14 "/HSPI_MISO")
 	(net 15 "/HSPI_CSO")
-	(net 16 "/L_TXD")
-	(net 17 "/L_RXD")
+	(net 16 "/U2_RX")
+	(net 17 "/U2_TX")
 	(net 18 "/LCD_SCK")
 	(net 19 "/LCD_SDA")
@@
 		(tags "resistor handsolder")
 		(property "Reference" "R7"
-			(at 2.556 0 -90)
+			(at 2.6545 0 -90)
 			(layer "F.SilkS")
 			(effects
@@
 		(descr "LED, diameter 3.0mm, 2 pins")
 		(tags "LED diameter 3.0mm 2 pins")
-		(property "Reference" "D3"
+		(property "Reference" "D1"
 			(at 3.937 -1.651 180)
 			(layer "F.SilkS")
@@
 			(layers "*.Cu" "*.Mask")
 			(remove_unused_layers no)
-			(net 21 "Net-(D3-A)")
+			(net 35 "Net-(D1-A)")
 			(pinfunction "A")
 			(pintype "passive")
@@
 			(layers "*.Cu" "*.Mask")
 			(remove_unused_layers no)
-			(net 17 "/L_RXD")
+			(net 17 "/U2_TX")
 			(pinfunction "Pin_2")
 			(pintype "passive")
@@
 			(layers "*.Cu" "*.Mask")
 			(remove_unused_layers no)
-			(net 16 "/L_TXD")
+			(net 16 "/U2_RX")
 			(pinfunction "Pin_3")
 			(pintype "passive")
@@
 			(size 1.5 0.9)
 			(layers "F.Cu" "F.Paste" "F.Mask")
-			(net 16 "/L_TXD")
+			(net 16 "/U2_RX")
 			(pinfunction "IO16")
 			(pintype "bidirectional")
@@
 			(size 1.5 0.9)
 			(layers "F.Cu" "F.Paste" "F.Mask")
-			(net 17 "/L_RXD")
+			(net 17 "/U2_TX")
 			(pinfunction "IO17")
 			(pintype "bidirectional")
@@
 		(descr "LED, diameter 3.0mm, 2 pins")
 		(tags "LED diameter 3.0mm 2 pins")
-		(property "Reference" "D1"
+		(property "Reference" "D3"
 			(at 3.937 -1.651 180)
 			(layer "F.SilkS")
@@
 			(layers "*.Cu" "*.Mask")
 			(remove_unused_layers no)
-			(net 35 "Net-(D1-A)")
+			(net 21 "Net-(D3-A)")
 			(pinfunction "A")
 			(pintype "passive")
@@
 		)
 		(property "Value" "JBAT"
-			(at 0 5.31 360)
+			(at 0 5.31 0)
 			(layer "F.Fab")
 			(effects
@@
 		(tags "Through hole socket strip THT 1x04 2.54mm single row")
 		(property "Reference" "J6"
-			(at -0.914 -1.651 270)
+			(at -0.914 -1.651 -90)
 			(layer "F.SilkS")
 			(effects
@@
 		)
 		(property "Value" "I2C"
-			(at 0 10.39 270)
+			(at 0 10.39 -90)
 			(layer "F.Fab")
 			(effects
@@
 		)
 		(fp_text user "${REFERENCE}"
-			(at 0 3.81 360)
+			(at 0 3.81 0)
 			(layer "F.Fab")
 			(effects
@@
 			(layers "*.Cu" "*.Mask")
 			(remove_unused_layers no)
-			(net 17 "/L_RXD")
+			(net 17 "/U2_TX")
 			(pinfunction "Pin_2")
 			(pintype "passive")
@@
 			(layers "*.Cu" "*.Mask")
 			(remove_unused_layers no)
-			(net 16 "/L_TXD")
+			(net 16 "/U2_RX")
 			(pinfunction "Pin_3")
 			(pintype "passive")
@@
 			(layers "B.Cu" "B.Paste" "B.Mask")
 			(roundrect_rratio 0.208333)
-			(net 35 "Net-(D1-A)")
+			(net 21 "Net-(D3-A)")
 			(pintype "passive")
 		)
@@
 		(tags "capacitor handsolder")
 		(property "Reference" "C17"
-			(at 3.1535 0 360)
+			(at 3.1535 0 0)
 			(layer "B.SilkS")
 			(effects
@@
 		)
 		(property "Value" "22uF"
-			(at 0 -1.68 360)
+			(at 0 -1.68 0)
 			(layer "B.Fab")
 			(effects
@@
 		)
 		(fp_text user "${REFERENCE}"
-			(at 0 0 360)
+			(at 0 0 0)
 			(layer "B.Fab")
 			(effects
@@
 			(layers "B.Cu" "B.Paste" "B.Mask")
 			(roundrect_rratio 0.208333)
-			(net 21 "Net-(D3-A)")
+			(net 35 "Net-(D1-A)")
 			(pintype "passive")
 		)
@@
 		(tags "capacitor handsolder")
 		(property "Reference" "C18"
-			(at 3.1535 0 360)
+			(at 3.1535 0 0)
 			(layer "B.SilkS")
 			(effects
@@
 		)
 		(property "Value" "22uF"
-			(at 0 -1.68 360)
+			(at 0 -1.68 0)
 			(layer "B.Fab")
 			(effects
@@
 		)
 		(fp_text user "${REFERENCE}"
-			(at 0 0 360)
+			(at 0 0 0)
 			(layer "B.Fab")
 			(effects
@@
 	(footprint "Capacitor_SMD:C_0805_2012Metric_Pad1.18x1.45mm_HandSolder"
 		(layer "B.Cu")
-		(at 147.32 83.82 -90)
+		(at 146.812 83.82 -90)
 		(descr "Capacitor SMD 0805 (2012 Metric), square (rectangular) end terminal, IPC_7351 nominal with elongated pad for handsoldering. (Body size source: IPC-SM-782 page 76, https://www.pcb-3d.com/wordpress/wp-content/uploads/ipc-sm-782a_amendment_1_and_2.pdf, https://docs.google.com/spreadsheets/d/1BsfQQcO9C6DZCsRaXUlFlo91Tg2WpOkGARC1WS5S8t0/edit?usp=sharing), generated with kicad-footprint-generator")
 		(tags "capacitor handsolder")
@@
 		)
 	)
+	(gr_text "XNS XSC XRS XIO2 GND"
+		(at 130.429 108.204 90)
+		(layer "F.SilkS")
+		(effects
+			(font
+				(size 0.75 0.75)
+				(thickness 0.1)
+			)
+			(justify left bottom)
+		)
+	)
+	(gr_text "5v XMI XMO XIO1 XIO0"
+		(at 124.079 107.696 90)
+		(layer "F.SilkS")
+		(effects
+			(font
+				(size 0.75 0.75)
+				(thickness 0.1)
+			)
+			(justify left bottom)
+		)
+	)
 	(gr_text "3v3  RX  TX  GND"
 		(at 114.554 125.476 0)
@@
 	)
 	(gr_text "Rádio"
-		(at 130.429 107.95 90)
+		(at 125.222 94.996 0)
 		(layer "F.SilkS")
 		(effects
@@
 		(layer "Dwgs.User")
 		(pts
+			(xy 149.86 81.28) (xy 106.68 81.28)
+		)
+		(height 3.683)
+		(gr_text "43.1800 mm"
+			(at 128.27 76.447 0)
+			(layer "Dwgs.User")
+			(effects
+				(font
+					(size 1 1)
+					(thickness 0.15)
+				)
+			)
+		)
+		(format
+			(prefix "")
+			(suffix "")
+			(units 3)
+			(units_format 1)
+			(precision 4)
+		)
+		(style
+			(thickness 0.1)
+			(arrow_length 1.27)
+			(text_position_mode 0)
+			(extension_height 0.58642)
+			(extension_offset 0.5) keep_text_aligned)
+	)
+	(dimension
+		(type aligned)
+		(layer "Dwgs.User")
+		(pts
+			(xy 106.68 81.28) (xy 106.68 124.46)
+		)
+		(height 14.351)
+		(gr_text "43.1800 mm"
+			(at 91.179 102.87 90)
+			(layer "Dwgs.User")
+			(effects
+				(font
+					(size 1 1)
+					(thickness 0.15)
+				)
+			)
+		)
+		(format
+			(prefix "")
+			(suffix "")
+			(units 3)
+			(units_format 1)
+			(precision 4)
+		)
+		(style
+			(thickness 0.1)
+			(arrow_length 1.27)
+			(text_position_mode 0)
+			(extension_height 0.58642)
+			(extension_offset 0.5) keep_text_aligned)
+	)
+	(dimension
+		(type aligned)
+		(layer "Dwgs.User")
+		(pts
 			(xy 158.6925 127.7335) (xy 158.6925 78.4575)
 		)
@@
 	)
 	(segment
-		(start 147.32 88.68)
+		(start 146.812 89.188)
 		(end 145.5 90.5)
 		(width 0.2032)
@@
 	)
 	(segment
-		(start 147.32 84.8575)
-		(end 147.32 88.68)
+		(start 146.812 84.8575)
+		(end 146.812 89.188)
 		(width 0.2032)
 		(layer "B.Cu")
@@
 	)
 	(segment
-		(start 117.348 96.647)
-		(end 119.253 96.647)
+		(start 117.226 101.219)
+		(end 119.258 101.219)
 		(width 0.1778)
 		(layer "B.Cu")
@@
 	)
 	(segment
-		(start 117.226 101.219)
-		(end 119.258 101.219)
+		(start 117.348 96.647)
+		(end 119.253 96.647)
 		(width 0.1778)
 		(layer "B.Cu")

Commit message: Update RiMon.kicad_pcb
Parts:
- moved D2 0.25 mm to (121.8, 106.0)
- moved D3 0.25 mm to (121.8, 101.5)
- moved R13 0.25 mm to (116.3, 106.0)
- moved R14 0.25 mm to (116.2, 101.5)
- moved D1 0.25 mm to (121.8, 96.9)
- moved R15 0.25 mm to (116.3, 96.9)
- moved C18 0.21 mm to (119.4, 115.8)
Routing:
- net /IO0: track 62.2 -> 58.9 mm
- net /EN: track 49.2 -> 51.0 mm
- net GND: vias 30 -> 40

Commit message: Finaliza Design
Parts:
- moved C20 2.21 mm to (103.3, 111.7), turned to -90 degrees
- moved C22 2.13 mm to (105.4, 111.2), turned to -90 degrees
Routing:
- net +5V: track 127.9 -> 138.3 mm, vias 3 -> 4
- net GND: track 6.01 -> 3.68 mm, vias 40 -> 42
- net /LED_Status: track 22.8 -> 21.5 mm
- net /IO0: track 58.9 -> 59.8 mm

Commit message: Ajustes fabricação
Parts:
- moved J10 0.20 mm to (145.5, 90.3)
Connections:
- J10 pad 6: unconnected-(J10-Pin_6-Pad6) -> GND
Routing:
- net GND: track 3.68 -> 16.7 mm
- net /HSPI_MOSI: track 12.6 -> 13.2 mm
Other:
- board size 63.2 x 49.3 mm -> 61.7 x 49.3 mm
- board text added: "COM"
- board text added: "MOSI MISO GND IO4 VN"
- board text added: "PWR"
- board text added: "STATUS"
- board text added: "vBat 12v"
- board text removed: "MOSI MISO 12vS IO4 VN"
